Commit message: Added ground utility function. TODO(jeh15): OSC on foot. Verify SAP constraints are ok.

File: models/digit_old.urdf (robot description, URDF)
Before this commit: robot digit, 35 links, 35 joints
Links:
- added link left-achilles-rod_link; collision capsule length=0.25 radius=0.007; visual mesh filename=obj/achilles-rod.obj
- added link left-toe-A-rod_link, mass 0.090983; collision capsule length=0.17 radius=0.007; visual mesh filename=obj/toe-A-rod.obj
- added link left-toe-A_visual, mass 0; visual sphere radius=0.02
- added link left-toe-B-rod_link, mass 0.079507; collision capsule length=0.144 radius=0.007; visual mesh filename=obj/toe-B-rod.obj
- added link right-achilles-rod_link; collision capsule length=0.25 radius=0.007; visual mesh filename=obj/achilles-rod.obj
- added link right-toe-A-rod_link, mass 0.090983; collision capsule length=0.17 radius=0.007; visual mesh filename=obj/toe-a-rod-xz.obj
- added link right-toe-B-rod_link, mass 0.079507; collision capsule length=0.144 radius=0.007; visual mesh filename=obj/toe-B-rod-xz.obj
- link left-elbow_link: geometry collision cylinder length=0.1565 radius=0.013; collision sphere radius=0.015
- link left-shoulder-pitch_link: geometry collision cylinder length=0.07 radius=0.038; visual mesh filename=obj/arm-L2.obj
- link left-shoulder-roll_link: geometry visual mesh filename=obj/arm-L1.obj
- link left-shoulder-yaw_link: geometry collision cylinder length=0.04 radius=0.03; collision cylinder length=0.0675 radius=0.038
- link right-elbow_link: geometry collision cylinder length=0.1565 radius=0.013; collision sphere radius=0.015
- link right-shoulder-pitch_link: geometry collision cylinder length=0.07 radius=0.038; visual mesh filename=obj/arm-L2-xz.obj
- link right-shoulder-roll_link: geometry visual mesh filename=obj/arm-L1-xz.obj
- link right-shoulder-yaw_link: geometry collision cylinder length=0.04 radius=0.03; collision cylinder length=0.0675 radius=0.038
Joints:
- added joint left-toe-A_visual_joint: type fixed, parent left-toe-A_link, child left-toe-A_visual, origin xyz=0.057 0 -0.008 rpy=0.005934119 0.03735005 -1.5437437
- joint base_joint: origin xyz=0 0 0 rpy=0 0 0 -> xyz=0 0 0 rpy=-0 0 -0
- joint left-shin_joint: type fixed -> continuous
- joint right-shin_joint: type fixed -> continuous
