Commit message: Fixed incorrect joint type in digit_open.urdf. Added more utilities.

File: models/digit_open.urdf (robot description, URDF)
Before this commit: robot digit, 35 links, 35 joints
Joints:
- joint left-shin_joint: type continuous -> fixed
- joint right-shin_joint: type continuous -> fixed

Commit message: Updated URDF

File: models/digit_open.urdf (robot description, URDF)
Before this commit: robot digit, 35 links, 35 joints
Links:
- link left-elbow_link: geometry collision cylinder length=0.1565 radius=0.013; collision sphere radius=0.015
- link left-shoulder-pitch_link: geometry collision cylinder length=0.07 radius=0.038; visual mesh filename=obj/arm-l2.obj
- link left-shoulder-roll_link: geometry visual mesh filename=obj/arm-l1.obj
- link left-shoulder-yaw_link: geometry collision cylinder length=0.04 radius=0.03; collision cylinder length=0.0675 radius=0.038
- link right-elbow_link: geometry collision cylinder length=0.1565 radius=0.013; collision sphere radius=0.015
- link right-shoulder-pitch_link: geometry collision cylinder length=0.07 radius=0.038; visual mesh filename=obj/arm-l2-xz.obj
- link right-shoulder-roll_link: geometry visual mesh filename=obj/arm-l1-xz.obj
- link right-shoulder-yaw_link: geometry collision cylinder length=0.04 radius=0.03; collision cylinder length=0.0675 radius=0.038

Commit message: OSC implemented

File: models/digit_open.urdf (robot description, URDF)
Before this commit: robot digit, 35 links, 35 joints
Links:
- added link trajectory_link, mass 0; visual cylinder length=0.005 radius=0.2
Joints:
- added joint trajectory_joint: type fixed, parent world, child trajectory_link, origin xyz=0 0 0 rpy=0 0 0

Commit message: Leg OSC: Kinematic constraints are causing issues.

File: models/digit_open.urdf (robot description, URDF)
Before this commit: robot digit, 36 links, 36 joints
Links:
- link trajectory_link: geometry visual cylinder length=0.005 radius=0.1
