Commit message: Fixed digit urdf

File: models/digit_old_.urdf (robot description, URDF)
Before this commit: robot digit, 35 links, 35 joints
Joints:
- joint left-elbow_joint: origin xyz=0 -0.0385 0.185 rpy=1.5707963267948966 -0.3926990816987242 6.0084837121965e-17 -> xyz=0 -0.0385 0.185 rpy=1.5708 0 0
- joint left-foot_joint: origin xyz=0 -0.05456 -0.0315 rpy=-4.440892098500625e-16 -1.0471975511965976 -1.5707963267948961 -> xyz=0 -0.05456 -0.0315 rpy=-1.0472 0 -1.5708
- joint left-hand_joint: origin xyz=0.369 0 -0.07912 rpy=1.5707963267948963 0.17453292519943295 -4.2275625162475e-17 -> xyz=0.369 0 -0.07912 rpy=1.5708 0 -0.174533
- joint left-heel-spring_joint: origin xyz=-0.01766 -0.029456 0.00104 rpy=-0.06890726319112118 -0.03703539652316154 2.720717602917085 -> xyz=-0.01766 -0.029456 0.00104 rpy=0.07801622 0.005585054 2.719223
- joint left-hip-pitch_joint: origin xyz=0 0.004 0.068 rpy=-1.5707963267948966 -0.7853981633974483 3.141592653589793 -> xyz=0 0.004 0.068 rpy=1.5708 0 0
- joint left-hip-roll_joint: origin xyz=-0.001 0.091 0 rpy=1.570796326794897 -1.1955505376161157 -1.570796326794897 -> xyz=-0.001 0.091 0 rpy=0 -1.5708 0
- joint left-hip-yaw_joint: origin xyz=-0.0505 0 0.044 rpy=0.0 -1.5707963267948966 0.0 -> xyz=-0.0505 0 0.044 rpy=0 -1.5708 0
- joint left-knee_joint: origin xyz=0.12 0 0.0045 rpy=0.0 0.0 -1.5707963267948966 -> xyz=-0.085 0.085 0.0045 rpy=0 0 0.785398
- joint left-shoulder-pitch_joint: origin xyz=-0.00317 -0.011055 0.0555 rpy=1.5707963267948966 0.7853981633974485 -0.2792526803190933 -> xyz=-0.00317 -0.011055 0.0555 rpy=1.5708 0 -0.279253
- joint left-shoulder-roll_joint: origin xyz=-0.001 0.12 0.4 rpy=-1.5707963267948954 -1.3962634015954636 1.5707963267948954 -> xyz=-0.001 0.12 0.4 rpy=-0.174533 -1.5708 0
- joint left-shoulder-yaw_joint: origin xyz=0 -0.165 -0.1 rpy=1.5707963267948966 -0.0 0.0 -> xyz=0 -0.165 -0.1 rpy=1.5708 0 0
- joint left-tarsus_joint: origin xyz=0.434759 0.02 0 rpy=0.0 -0.0 1.7976891295541595 -> xyz=0.434759 0.02 0 rpy=0 0 1.79769
- joint left-toe-A_joint: origin xyz=0.059 -0.034 -0.0276 rpy=-3.141592653589793 1.2244450599234578e-16 -1.5526449025741558 -> xyz=0.059 -0.034 -0.0276 rpy=-3.14159 0 -1.5526449
- joint left-toe-B_joint: origin xyz=0.111 -0.034 0.0276 rpy=0.0 0.0 -1.5526449025741558 -> xyz=0.111 -0.034 0.0276 rpy=0 0 -1.5526449
- joint left-toe-pitch_joint: origin xyz=0.408 -0.04 0 rpy=0.0 -0.0 1.2522737383059317 -> xyz=0.408 -0.04 0 rpy=0 0 1.2522737
- joint left-toe-roll_joint: origin xyz=0 0 0 rpy=-0.0 1.5707963267948966 0.0 -> xyz=0 0 0 rpy=0 1.5708 0
- joint right-elbow_joint: origin xyz=0 0.0385 0.185 rpy=-1.5707963267948966 -0.3926990816987242 -6.0084837121965e-17 -> xyz=0 0.0385 0.185 rpy=-1.5708 0 0
- joint right-foot_joint: origin xyz=0 0.05456 -0.0315 rpy=4.440892098500625e-16 -1.0471975511965976 1.5707963267948961 -> xyz=0 0.05456 -0.0315 rpy=1.0472 0 1.5708
- joint right-hand_joint: origin xyz=0.369 0 -0.07912 rpy=-1.5707963267948963 0.17453292519943295 4.2275625162475e-17 -> xyz=0.369 0 -0.07912 rpy=-1.5708 0 0.174533
- joint right-heel-spring_joint: origin xyz=-0.01766 0.029456 0.00104 rpy=0.06890726319112118 -0.03703539652316154 -2.720717602917085 -> xyz=-0.01766 0.029456 0.00104 rpy=-0.07801622 0.005585054 -2.719223
- joint right-hip-pitch_joint: origin xyz=0 -0.004 0.068 rpy=1.5707963267948966 -0.7853981633974483 -3.141592653589793 -> xyz=0 -0.004 0.068 rpy=-1.5708 0 0
- joint right-hip-roll_joint: origin xyz=-0.001 -0.091 0 rpy=-1.570796326794897 -1.1955505376161157 1.570796326794897 -> xyz=-0.001 -0.091 0 rpy=0 -1.5708 0
- joint right-hip-yaw_joint: origin xyz=-0.0505 0 0.044 rpy=0.0 -1.5707963267948966 0.0 -> xyz=-0.0505 0 0.044 rpy=0 -1.5708 0
- joint right-knee_joint: origin xyz=0.12 0 0.0045 rpy=0.0 -0.0 1.5707963267948966 -> xyz=-0.085 -0.085 0.0045 rpy=0 0 -0.785398
- joint right-shoulder-pitch_joint: origin xyz=-0.00317 0.011055 0.0555 rpy=-1.5707963267948966 0.7853981633974485 0.2792526803190933 -> xyz=-0.00317 0.011055 0.0555 rpy=-1.5708 0 0.279253
- joint right-shoulder-roll_joint: origin xyz=-0.001 -0.12 0.4 rpy=1.5707963267948954 -1.3962634015954636 -1.5707963267948954 -> xyz=-0.001 -0.12 0.4 rpy=0.174533 -1.5708 0
- joint right-shoulder-yaw_joint: origin xyz=0 0.165 -0.1 rpy=-1.5707963267948966 0.0 0.0 -> xyz=0 0.165 -0.1 rpy=-1.5708 0 0
- joint right-tarsus_joint: origin xyz=0.434759 -0.02 0 rpy=0.0 0.0 -1.7976891295541595 -> xyz=0.434759 -0.02 0 rpy=0 0 -1.79769
- joint right-toe-A_joint: origin xyz=0.059 0.034 -0.0276 rpy=3.141592653589793 1.2244450599234578e-16 1.5526449025741558 -> xyz=0.059 0.034 -0.0276 rpy=3.14159 0 1.5526449
- joint right-toe-B_joint: origin xyz=0.111 0.034 0.0276 rpy=0.0 -0.0 1.5526449025741558 -> xyz=0.111 0.034 0.0276 rpy=0 0 1.5526449
- joint right-toe-pitch_joint: origin xyz=0.408 0.04 0 rpy=0.0 0.0 -1.2522737383059317 -> xyz=0.408 0.04 0 rpy=0 0 -1.2522737
- joint right-toe-roll_joint: origin xyz=0 0 0 rpy=-0.0 1.5707963267948966 0.0 -> xyz=0 0 0 rpy=0 1.5708 0
