Commit message: Updated URDF

File: models/digit.urdf (robot description, URDF)
Before this commit: robot digit, 41 links, 35 joints
Links:
- added link left-toe-A_visual, mass 0; visual sphere radius=0.02
Joints:
- added joint left-toe-A_visual_joint: type fixed, parent left-toe-A_link, child left-toe-A_visual, origin xyz=0.057 0 -0.008 rpy=0.005934119 0.03735005 -1.5437437

Commit message: Pushing local changes. Messy need to refactor. TODO: Test feet motors.

File: models/digit.urdf (robot description, URDF)
Before this commit: robot digit, 35 links, 35 joints
Links:
- link right-hip-yaw_link: geometry visual cylinder length=0.1 radius=0.01; visual cylinder length=0.1 radius=0.01

Commit message: Added zero moment constraint. TODO: refactor.

File: models/digit.urdf (robot description, URDF)
Before this commit: robot digit, 35 links, 35 joints
Links:
- link right-hip-yaw_link: geometry visual mesh filename=obj/hip-pitch-housing-xz.obj
